File: KiCad_src/CW312T_STM32F.kicad_pcb (KiCad board)
At the start: 2 copper layers, 58.7 x 48.7 mm, 35 parts, among them J1 USB_C, P1 PCIeX4-GF-2D-1000-1K-O64, U1 USBLC6-2SC6, U2 STM32F405VGT6

Commit message: Updated
Parts:
- NT10, NT11, NT2, NT3, NT7, NT9: moved to B.Cu
- moved NT3 34.8 mm to (167.6, 83.0), turned to 90 degrees
- moved NT2 34.4 mm to (165.6, 83.0), turned to 90 degrees
- moved NT11 31.9 mm to (169.0, 85.4)
- moved C14 31.4 mm to (174.3, 112.5), turned to -90 degrees
- moved NT1 29.7 mm to (165.0, 108.1), turned to -90 degrees
- moved NT8 28.8 mm to (166.6, 82.9), turned to -90 degrees
- moved NT10 27.0 mm to (164.2, 85.4)
- moved NT9 20.3 mm to (157.0, 85.4)
- moved R4 16.1 mm to (145.2, 100.7), turned to 90 degrees
- moved C2 14.9 mm to (150.5, 90.4), turned to 90 degrees
- moved R6 13.7 mm to (156.5, 90.4), turned to 90 degrees
- moved C12 9.49 mm to (171.5, 108.5), turned to 90 degrees
- moved C10 8.65 mm to (172.1, 101.7), turned to -90 degrees
- moved NT7 7.87 mm to (143.6, 83.0), turned to -90 degrees
- moved C13 3.68 mm to (171.5, 112.5), turned to -90 degrees
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Connections:
- NT8 pad 2: JTAG_VREF -> HDR2
Routing:
- net +3V3: track 11.8 -> 29.6 mm
- net HDR4: track 0.00 -> 11.9 mm
- net HDR2: track 0.00 -> 9.55 mm, vias 0 -> 1
- net FILTIN: track 0.00 -> 4.84 mm
- net +1V2: track 0.00 -> 4.82 mm
- net GND: track 0.00 -> 4.03 mm, vias 0 -> 2
- net CW_PDIC/BOOT0: track 0.00 -> 3.65 mm
- net JTAG_nRST: track 0.00 -> 3.03 mm
- net HDR3: track 0.00 -> 3.03 mm
- net HDR1: track 0.00 -> 3.03 mm
- net IOVREF: track 0.00 -> 2.93 mm
- net Net-(J1-D+-PadA6): track 15.3 -> 17.1 mm
- net Net-(J1-D--PadA7): track 17.9 -> 19.4 mm
- net +5V: track 15.2 -> 16.4 mm
