File: KiCad_src/CW312T_STM32F.kicad_sch (KiCad schematic)
At the start: 35 parts, among them J1 USB_C, P1 PCIeX4-GF-2D-1000-1K-O64, U1 USBLC6-2SC6, U2 STM32F405VGT6

Commit message: Updated
Connections:
- net HDR2: now also NT8.2
- net JTAG_VREF: no longer NT8.2
Changed lines of the file:
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@@
 	)
 	(junction
-		(at 257.81 21.59)
-		(diameter 0)
-		(color 0 0 0 0)
-	)
-	(junction
 		(at 129.54 21.59)
 		(diameter 0)
@@
 	(wire
 		(pts
+			(xy 267.97 19.05) (xy 267.97 21.59)
+		)
+		(stroke
+			(width 0)
+			(type default)
+		)
+	)
+	(wire
+		(pts
 			(xy 246.38 58.42) (xy 248.92 58.42)
 		)
@@
 	(wire
 		(pts
+			(xy 257.81 19.05) (xy 267.97 19.05)
+		)
+		(stroke
+			(width 0)
+			(type default)
+		)
+	)
+	(wire
+		(pts
 			(xy 246.38 127) (xy 248.92 127)
 		)
@@
 	(wire
 		(pts
+			(xy 252.73 19.05) (xy 252.73 24.13)
+		)
+		(stroke
+			(width 0)
+			(type default)
+		)
+	)
+	(wire
+		(pts
 			(xy 21.59 119.38) (xy 21.59 120.65)
 		)
@@
 	(wire
 		(pts
-			(xy 252.73 24.13) (xy 252.73 21.59)
-		)
-		(stroke
-			(width 0)
-			(type default)
-		)
-	)
-	(wire
-		(pts
 			(xy 132.08 172.72) (xy 132.08 175.26)
 		)
@@
 	(symbol
 		(lib_id "Device:NetTie_2")
-		(at 255.27 21.59 0)
+		(at 255.27 19.05 0)
 		(unit 1)
 		(body_style 1)
@@
 		(fields_autoplaced yes)
 		(property "Reference" "NT8"
-			(at 255.27 16.51 0)
+			(at 255.27 13.97 0)
 			(hide yes)
 			(show_name no)
@@
 		)
 		(property "Value" "NetTie_2"
-			(at 255.27 19.05 0)
+			(at 255.27 16.51 0)
 			(hide yes)
 			(show_name no)
@@
 		)
 		(property "Footprint" "NetTie:NetTie-2_SMD_Pad0.5mm"
-			(at 255.27 21.59 0)
+			(at 255.27 19.05 0)
 			(hide yes)
 			(show_name no)
@@
 		)
 		(property "Datasheet" ""
-			(at 255.27 21.59 0)
+			(at 255.27 19.05 0)
 			(hide yes)
 			(show_name no)
@@
 		)
 		(property "Description" "Net tie, 2 pins"
-			(at 255.27 21.59 0)
+			(at 255.27 19.05 0)
 			(hide yes)
 			(show_name no)
